Commit message: Fix per-robot topic namespacing (botname in LIDAR/DiffDrive topics), add missing Sensors plugin, fix missing closing robot tag; add MAPPO algorithm notes and marl_training scripts

File: src/jetbot_description/urdf/jetbot.urdf.xacro (robot description, xacro)
@@ -1,4 +1,6 @@
 <?xml version="1.0"?>
 <robot name="jetbot" xmlns:xacro="http://www.ros.org/wiki/xacro">
+  <xacro:arg name="botname" default="jetbot"/>
+  <xacro:property name="botname" value="$(arg botname)"/>
   <!-- ===================== Base ===================== -->
   <link name="base_link">
@@ -138,5 +140,5 @@
       <wheel_radius>0.033</wheel_radius>
       <odom_publish_frequency>30</odom_publish_frequency>
-      <topic>cmd_vel</topic>
+      <topic>${botname}/cmd_vel</topic>
     </plugin>
     <plugin filename="gz-sim-pose-publisher-system" name="gz::sim::systems::PosePublisher">
@@ -148,5 +150,5 @@
   <gazebo reference="lidar_link">
     <sensor name="lidar" type="gpu_lidar">
-      <topic>scan</topic>
+      <topic>${botname}/scan</topic>
       <update_rate>5.5</update_rate>
       <lidar>
